File: HDMI_to_Stemma/15Pin_Fanout/15Pin_Fanout/15Pin_Fanout.kicad_sch (KiCad schematic)
At the start: 7 parts, among them J1 HDMI_A, J2 Conn_01x02, J3 Conn_01x02, J4 Conn_01x02, J5 Conn_01x02, J6 Conn_01x04, J7 Conn_01x04

Commit message: Update
Parts:
- J1: LCSC (none) -> C111617
Changed lines of the file:
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@@
+      (effects (font (size 1.27 1.27)) hide)
+    )
+    (property "LCSC" "C111617" (id 4) (at 116.459 71.12 0)
       (effects (font (size 1.27 1.27)) hide)
     )
