File: HDMI_to_Stemma/15Pin_Fanout _Diodes_&_Heater/15Pin_Fanout/15Pin_Fanout.kicad_pcb (KiCad board)
At the start: 2 copper layers, 25 x 30.5 mm, 4 parts, among them J1 HDMI_A, J2 Conn_01x02, J3 Conn_01x02, J6 Conn_01x04

Commit message: Update
Routing:
- net GND: track 16.7 -> 17.8 mm, vias 0 -> 1
Other:
- board text added: "HDMI_JST_15Pin_Diodes & Heater Ryan Morgenstern 6/62022"
- board text removed: "HDMI_JST_15Pin_Diodes Ryan Morgenstern 6/62022"
Changed lines of the file:
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@@
       (drillshape 0)
       (scaleselection 1)
-      (outputdirectory "C:/Users/rdm8/Documents/GitHub/MicroD_Stemma_Fanout/HDMI_to_Stemma/15Pin_Fanout _Diodes_&_Heater/15Pin_Fanout/Gerber/")
+      (outputdirectory "Gerber/")
     )
   )
@@
   (gr_line (start -8.5 -15) (end -12.5 -15) (layer "Edge.Cuts") (width 0.1))
   (gr_line (start 8.5 -5) (end 8.5 -15) (layer "Edge.Cuts") (width 0.1))
-  (gr_text "HDMI_JST_15Pin_Diodes\nRyan Morgenstern\n6/62022" (at -4.25 -7.25 90) (layer "B.SilkS")
+  (gr_text "HDMI_JST_15Pin_Diodes & Heater\nRyan Morgenstern\n6/62022" (at -2.75 -7.75 90) (layer "B.SilkS")
     (effects (font (size 1 1) (thickness 0.15)) (justify mirror))
   )
@@
   (segment (start 7.8 -17.139668) (end 7.8 -18.53) (width 0.25) (layer "F.Cu") (net 1))
   (segment (start -3.501 -1.946) (end -3.501 -3.396) (width 0.25) (layer "F.Cu") (net 2))
+  (segment (start -2.25 -1.74296) (end -2.25 -0.75) (width 0.25) (layer "F.Cu") (net 2))
   (segment (start 3.805 -1.75) (end 2.834323 -1.75) (width 0.25) (layer "F.Cu") (net 2))
   (segment (start 2.5 -1.946) (end 2.42548 -1.87148) (width 0.25) (layer "F.Cu") (net 2))
   (segment (start -0.5 -3.396) (end -0.5 -1.946) (width 0.25) (layer "F.Cu") (net 2))
   (segment (start 4.001 -3.396) (end 4.001 -1.946) (width 0.25) (layer "F.Cu") (net 2))
-  (segment (start -0.42548 -1.87148) (end -3.42648 -1.87148) (width 0.25) (layer "F.Cu") (net 2))
+  (segment (start -0.42548 -1.87148) (end -2.12148 -1.87148) (width 0.25) (layer "F.Cu") (net 2))
   (segment (start 2.834323 -1.75) (end 2.5 -2.084323) (width 0.25) (layer "F.Cu") (net 2))
   (segment (start 2.5 -2.084323) (end 2.5 -3.396) (width 0.25) (layer "F.Cu") (net 2))
   (segment (start -0.5 -1.946) (end -0.42548 -1.87148) (width 0.25) (layer "F.Cu") (net 2))
+  (segment (start -2.12148 -1.87148) (end -3.42648 -1.87148) (width 0.25) (layer "F.Cu") (net 2))
   (segment (start -0.42548 -1.87148) (end 1.313803 -1.87148) (width 0.25) (layer "F.Cu") (net 2))
   (segment (start 4.001 -1.946) (end 3.805 -1.75) (width 0.25) (layer "F.Cu") (net 2))
@@
   (segment (start -3.42648 -1.87148) (end -3.501 -1.946) (width 0.25) (layer "F.Cu") (net 2))
   (segment (start 1 -2.185283) (end 1 -3.396) (width 0.25) (layer "F.Cu") (net 2))
+  (segment (start -2.12148 -1.87148) (end -2.25 -1.74296) (width 0.25) (layer "F.Cu") (net 2))
+  (via (at -2.25 -0.75) (size 0.8) (drill 0.4) (layers "F.Cu" "B.Cu") (net 2))
   (segment (start 3.501 -13.476386) (end 6.8 -16.775386) (width 0.25) (layer "F.Cu") (net 3))
   (segment (start 6.8 -16.775386) (end 6.8 -18.53) (width 0.25) (layer "F.Cu") (net 3))

Commit message: Updated traces
Routing:
- net GND: track 17.8 -> 23.6 mm, vias 1 -> 5
- net Net-(J1-Pad12): track 16.8 -> 18.1 mm
- net Net-(J1-Pad1): track 16.5 -> 17.1 mm
Changed lines of the file:
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@@
     (effects (font (size 1 1) (thickness 0.15)) (justify mirror))
   )
+  (segment (start 4.525614 -8.749) (end 5.224511 -8.050103) (width 0.25) (layer "F.Cu") (net 1))
+  (segment (start 5.224511 -4.119511) (end 4.501 -3.396) (width 0.25) (layer "F.Cu") (net 1))
   (segment (start 4.501 -13.840668) (end 7.8 -17.139668) (width 0.25) (layer "F.Cu") (net 1))
-  (segment (start 4.501 -3.396) (end 4.501 -13.840668) (width 0.25) (layer "F.Cu") (net 1))
+  (segment (start 5.224511 -8.050103) (end 5.224511 -4.119511) (width 0.25) (layer "F.Cu") (net 1))
+  (segment (start 4.501 -13.840668) (end 4.501 -8.749) (width 0.25) (layer "F.Cu") (net 1))
   (segment (start 7.8 -17.139668) (end 7.8 -18.53) (width 0.25) (layer "F.Cu") (net 1))
-  (segment (start -3.501 -1.946) (end -3.501 -3.396) (width 0.25) (layer "F.Cu") (net 2))
-  (segment (start -2.25 -1.74296) (end -2.25 -0.75) (width 0.25) (layer "F.Cu") (net 2))
-  (segment (start 3.805 -1.75) (end 2.834323 -1.75) (width 0.25) (layer "F.Cu") (net 2))
-  (segment (start 2.5 -1.946) (end 2.42548 -1.87148) (width 0.25) (layer "F.Cu") (net 2))
-  (segment (start -0.5 -3.396) (end -0.5 -1.946) (width 0.25) (layer "F.Cu") (net 2))
-  (segment (start 4.001 -3.396) (end 4.001 -1.946) (width 0.25) (layer "F.Cu") (net 2))
-  (segment (start -0.42548 -1.87148) (end -2.12148 -1.87148) (width 0.25) (layer "F.Cu") (net 2))
-  (segment (start 2.834323 -1.75) (end 2.5 -2.084323) (width 0.25) (layer "F.Cu") (net 2))
-  (segment (start 2.5 -2.084323) (end 2.5 -3.396) (width 0.25) (layer "F.Cu") (net 2))
-  (segment (start -0.5 -1.946) (end -0.42548 -1.87148) (width 0.25) (layer "F.Cu") (net 2))
-  (segment (start -2.12148 -1.87148) (end -3.42648 -1.87148) (width 0.25) (layer "F.Cu") (net 2))
-  (segment (start -0.42548 -1.87148) (end 1.313803 -1.87148) (width 0.25) (layer "F.Cu") (net 2))
-  (segment (start 4.001 -1.946) (end 3.805 -1.75) (width 0.25) (layer "F.Cu") (net 2))
-  (segment (start 1.313803 -1.87148) (end 1 -2.185283) (width 0.25) (layer "F.Cu") (net 2))
-  (segment (start 2.42548 -1.87148) (end 1.313803 -1.87148) (width 0.25) (layer "F.Cu") (net 2))
-  (segment (start 2.5 -3.396) (end 2.5 -1.946) (width 0.25) (layer "F.Cu") (net 2))
-  (segment (start -3.42648 -1.87148) (end -3.501 -1.946) (width 0.25) (layer "F.Cu") (net 2))
-  (segment (start 1 -2.185283) (end 1 -3.396) (width 0.25) (layer "F.Cu") (net 2))
-  (segment (start -2.12148 -1.87148) (end -2.25 -1.74296) (width 0.25) (layer "F.Cu") (net 2))
-  (via (at -2.25 -0.75) (size 0.8) (drill 0.4) (layers "F.Cu" "B.Cu") (net 2))
+  (segment (start 4.501 -8.749) (end 4.525614 -8.749) (width 0.25) (layer "F.Cu") (net 1))
+  (segment (start 4.001 -7.251) (end 4.001 -3.396) (width 0.25) (layer "F.Cu") (net 2))
+  (segment (start 4.001 -7.251) (end 4.5 -7.75) (width 0.25) (layer "F.Cu") (net 2))
+  (segment (start 1 -3.396) (end 1 -10.2755) (width 0.25) (layer "F.Cu") (net 2))
+  (segment (start 1 -10.2755) (end 1.2245 -10.5) (width 0.25) (layer "F.Cu") (net 2))
+  (segment (start -0.5 -3.396) (end -0.5 -5.75) (width 0.25) (layer "F.Cu") (net 2))
+  (segment (start -3.501 -3.396) (end -3.501 -5.249) (width 0.25) (layer "F.Cu") (net 2))
+  (segment (start -0.5 -5.75) (end -1.75 -7) (width 0.25) (layer "F.Cu") (net 2))
+  (segment (start -3.501 -5.249) (end -3.5 -5.25) (width 0.25) (layer "F.Cu") (net 2))
+  (segment (start 2.5 -8.945785) (end 2.7245 -9.170285) (width 0.25) (layer "F.Cu") (net 2))
+  (segment (start 2.5 -3.396) (end 2.5 -8.945785) (width 0.25) (layer "F.Cu") (net 2))
+  (via (at -1.75 -7) (size 0.8) (drill 0.4) (layers "F.Cu" "B.Cu") (net 2))
+  (via (at 2.7245 -9.170285) (size 0.8) (drill 0.4) (layers "F.Cu" "B.Cu") (net 2))
+  (via (at 1.2245 -10.5) (size 0.8) (drill 0.4) (layers "F.Cu" "B.Cu") (net 2))
+  (via (at -3.5 -5.25) (size 0.8) (drill 0.4) (layers "F.Cu" "B.Cu") (net 2))
+  (via (at 4.5 -7.75) (size 0.8) (drill 0.4) (layers "F.Cu" "B.Cu") (net 2))
+  (segment (start 3.898531 -13.078855) (end 3.501 -13.476386) (width 0.25) (layer "F.Cu") (net 3))
+  (segment (start 3.501 -8.286453) (end 3.898531 -8.683984) (width 0.25) (layer "F.Cu") (net 3))
   (segment (start 3.501 -13.476386) (end 6.8 -16.775386) (width 0.25) (layer "F.Cu") (net 3))
   (segment (start 6.8 -16.775386) (end 6.8 -18.53) (width 0.25) (layer "F.Cu") (net 3))
-  (segment (start 3.501 -3.396) (end 3.501 -13.476386) (width 0.25) (layer "F.Cu") (net 3))
+  (segment (start 3.898531 -8.683984) (end 3.898531 -13.078855) (width 0.25) (layer "F.Cu") (net 3))
+  (segment (start 3.501 -3.396) (end 3.501 -8.286453) (width 0.25) (layer "F.Cu") (net 3))
+  (segment (start 2.89904 -10.5) (end 2.89904 -13.89904) (width 0.25) (layer "F.Cu") (net 4))
+  (segment (start 2.89904 -13.89904) (end 3 -14) (width 0.25) (layer "F.Cu") (net 4))
   (segment (start 3.001 -13.999) (end 3 -14) (width 0.25) (layer "F.Cu") (net 4))
+  (segment (start 3.001 -3.396) (end 3.001 -8.422171) (width 0.25) (layer "F.Cu") (net 4))
+  (segment (start 3.001 -8.422171) (end 3.449011 -8.870182) (width 0.25) (layer "F.Cu") (net 4))
+  (segment (start 3.449011 -8.870182) (end 3.449011 -9.950029) (width 0.25) (layer "F.Cu") (net 4))
   (segment (start 9 -16.5) (end 9 -18.33) (width 0.25) (layer "F.Cu") (net 4))
   (segment (start 9 -18.33) (end 8.8 -18.53) (width 0.25) (layer "F.Cu") (net 4))
-  (segment (start 3.001 -3.396) (end 3.001 -13.999) (width 0.25) (layer "F.Cu") (net 4))
+  (segment (start 3.449011 -9.950029) (end 2.89904 -10.5) (width 0.25) (layer "F.Cu") (net 4))
   (via (at 3 -14) (size 0.8) (drill 0.4) (layers "F.Cu" "B.Cu") (net 4))
   (via (at 9 -16.5) (size 0.8) (drill 0.4) (layers "F.Cu" "B.Cu") (net 4))
   (segment (start 6.5 -14) (end 9 -16.5) (width 0.25) (layer "B.Cu") (net 4))
   (segment (start 3 -14) (end 6.5 -14) (width 0.25) (layer "B.Cu") (net 4))
-  (segment (start 2 -14.73) (end 5.8 -18.53) (width 0.25) (layer "F.Cu") (net 5))
-  (segment (start 2 -3.396) (end 2 -14.73) (width 0.25) (layer "F.Cu") (net 5))
+  (segment (start 2.01 -14.74) (end 5.8 -18.53) (width 0.25) (layer "F.Cu") (net 5))
+  (segment (start 2.44952 -10.064688) (end 2.44952 -11) (width 0.25) (layer "F.Cu") (net 5))
+  (segment (start 2.01 -11.43952) (end 2.01 -14.74) (width 0.25) (layer "F.Cu") (net 5))
+  (segment (start 2 -14.73) (end 2.01 -14.74) (width 0.25) (layer "F.Cu") (net 5))
+  (segment (start 2.44952 -11) (end 2.01 -11.43952) (width 0.25) (layer "F.Cu") (net 5))
+  (segment (start 2 -3.396) (end 2 -9.615168) (width 0.25) (layer "F.Cu") (net 5))
+  (segment (start 2 -9.615168) (end 2.44952 -10.064688) (width 0.25) (layer "F.Cu") (net 5))
+  (segment (start 1.5 -9.749114) (end 1.5 -3.396) (width 0.25) (layer "F.Cu") (net 6))
+  (segment (start 1.5 -16.25) (end 1.5 -11.249114) (width 0.25) (layer "F.Cu") (net 6))
   (segment (start 0.65 -17.1) (end 1.5 -16.25) (width 0.25) (layer "F.Cu") (net 6))
-  (segment (start 1.5 -16.25) (end 1.5 -3.396) (width 0.25) (layer "F.Cu") (net 6))
+  (segment (start 2 -10.250886) (end 1.499114 -9.75) (width 0.25) (layer "F.Cu") (net 6))
+  (segment (start 2 -10.749114) (end 2 -10.250886) (width 0.25) (layer "F.Cu") (net 6))
+  (segment (start 1.499114 -9.75) (end 1.5 -9.749114) (width 0.25) (layer "F.Cu") (net 6))
+  (segment (start 1.5 -11.249114) (end 2 -10.749114) (width 0.25) (layer "F.Cu") (net 6))
   (segment (start -1.35 -17.1) (end 0.5 -15.25) (width 0.25) (layer "F.Cu") (net 7))
-  (segment (start 0.5 -15.25) (end 0.5 -3.396) (width 0.25) (layer "F.Cu") (net 7))
+  (segment (start 0.5 -3.396) (end 0.5 -15.25) (width 0.25) (layer "F.Cu") (net 7))
   (segment (start 0 -10.55) (end 0 -3.396) (width 0.25) (layer "F.Cu") (net 8))
   (segment (start -6.55 -17.1) (end 0 -10.55) (width 0.25) (layer "F.Cu") (net 8))
-  (segment (start -1 -9.55) (end -1 -3.396) (width 0.25) (layer "F.Cu") (net 9))
+  (segment (start -2.474511 -7.300103) (end -2.474511 -6.131708) (width 0.25) (layer "F.Cu") (net 9))
+  (segment (start -1 -9.55) (end -1 -8.774614) (width 0.25) (layer "F.Cu") (net 9))
   (segment (start -8.55 -17.1) (end -1 -9.55) (width 0.25) (layer "F.Cu") (net 9))
+  (segment (start -1 -8.774614) (end -2.474511 -7.300103) (width 0.25) (layer "F.Cu") (net 9))
+  (segment (start -1 -4.657197) (end -1 -3.396) (width 0.25) (layer "F.Cu") (net 9))
+  (segment (start -2.474511 -6.131708) (end -1 -4.657197) (width 0.25) (layer "F.Cu") (net 9))
   (zone (net 2) (net_name "GND") (layer "F.Cu") (hatch edge 0.508)
     (connect_pads (clearance 0.508))
