File: HDMI_to_Stemma/15Pin_Fanout_Diodes/15Pin_Fanout/15Pin_Fanout.kicad_pcb (KiCad board)
At the start: 2 copper layers, 17 x 28 mm, 3 parts, among them J1 HDMI_A, J6 Conn_01x04, J7 Conn_01x04

Commit message: Update
Routing:
- net GND: track 19.0 -> 19.9 mm, vias 0 -> 1
Changed lines of the file:
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@@
   (segment (start 1 -1.946) (end 0.92548 -1.87148) (width 0.25) (layer "F.Cu") (net 2))
   (segment (start 2.5 -2.186283) (end 2.5 -3.396) (width 0.25) (layer "F.Cu") (net 2))
+  (segment (start -3.42648 -1.87148) (end -2.62852 -1.87148) (width 0.25) (layer "F.Cu") (net 2))
   (segment (start -0.5 -2.185283) (end -0.5 -3.396) (width 0.25) (layer "F.Cu") (net 2))
+  (segment (start -2.62852 -1.87148) (end -2.62852 -1.12852) (width 0.25) (layer "F.Cu") (net 2))
   (segment (start -0.813803 -1.87148) (end -0.5 -2.185283) (width 0.25) (layer "F.Cu") (net 2))
   (segment (start 1 -3.396) (end 1 -1.946) (width 0.25) (layer "F.Cu") (net 2))
@@
   (segment (start 0.92548 -1.87148) (end -0.37148 -1.87148) (width 0.25) (layer "F.Cu") (net 2))
   (segment (start -3.501 -3.396) (end -3.501 -1.946) (width 0.25) (layer "F.Cu") (net 2))
-  (segment (start -3.42648 -1.87148) (end -0.813803 -1.87148) (width 0.25) (layer "F.Cu") (net 2))
+  (segment (start -2.62852 -1.87148) (end -0.813803 -1.87148) (width 0.25) (layer "F.Cu") (net 2))
+  (segment (start -2.62852 -1.12852) (end -2.5 -1) (width 0.25) (layer "F.Cu") (net 2))
   (segment (start -0.37148 -1.87148) (end -0.5 -2) (width 0.25) (layer "F.Cu") (net 2))
   (segment (start 1 -2.185283) (end 1 -3.396) (width 0.25) (layer "F.Cu") (net 2))
   (segment (start 4.001 -3.396) (end 4.001 -1.946) (width 0.25) (layer "F.Cu") (net 2))
   (segment (start 2.5 -3.396) (end 2.5 -1.946) (width 0.25) (layer "F.Cu") (net 2))
+  (via (at -2.5 -1) (size 0.8) (drill 0.4) (layers "F.Cu" "B.Cu") (net 2))
   (segment (start 3.501 -16.499) (end 3.501 -3.396) (width 0.25) (layer "F.Cu") (net 3))
   (segment (start 3.5 -16.5) (end 3.501 -16.499) (width 0.25) (layer "F.Cu") (net 3))

Commit message: Updated traces
Routing:
- net GND: track 19.9 -> 16.5 mm, vias 1 -> 5
- net Net-(J1-Pad7): track 15.2 -> 16.0 mm
- net Net-(J1-Pad1): track 13.1 -> 13.9 mm
Changed lines of the file:
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@@
     (effects (font (size 1 1) (thickness 0.15)) (justify mirror))
   )
+  (segment (start 5.474511 -12.750875) (end 4.5 -13.725386) (width 0.25) (layer "F.Cu") (net 1))
+  (segment (start 4.5 -13.725386) (end 4.5 -16.5) (width 0.25) (layer "F.Cu") (net 1))
   (segment (start 4.501 -16.499) (end 4.5 -16.5) (width 0.25) (layer "F.Cu") (net 1))
-  (segment (start 4.501 -3.396) (end 4.501 -16.499) (width 0.25) (layer "F.Cu") (net 1))
-  (segment (start 3.805 -1.75) (end 2.936283 -1.75) (width 0.25) (layer "F.Cu") (net 2))
-  (segment (start 2.936283 -1.75) (end 2.5 -2.186283) (width 0.25) (layer "F.Cu") (net 2))
-  (segment (start 1 -1.946) (end 0.92548 -1.87148) (width 0.25) (layer "F.Cu") (net 2))
-  (segment (start 2.5 -2.186283) (end 2.5 -3.396) (width 0.25) (layer "F.Cu") (net 2))
-  (segment (start -3.42648 -1.87148) (end -2.62852 -1.87148) (width 0.25) (layer "F.Cu") (net 2))
-  (segment (start -0.5 -2.185283) (end -0.5 -3.396) (width 0.25) (layer "F.Cu") (net 2))
-  (segment (start -2.62852 -1.87148) (end -2.62852 -1.12852) (width 0.25) (layer "F.Cu") (net 2))
-  (segment (start -0.813803 -1.87148) (end -0.5 -2.185283) (width 0.25) (layer "F.Cu") (net 2))
-  (segment (start 1 -3.396) (end 1 -1.946) (width 0.25) (layer "F.Cu") (net 2))
-  (segment (start -0.5 -2) (end -0.5 -3.396) (width 0.25) (layer "F.Cu") (net 2))
-  (segment (start 2.5 -1.946) (end 2.42548 -1.87148) (width 0.25) (layer "F.Cu") (net 2))
-  (segment (start 2.42548 -1.87148) (end 1.313803 -1.87148) (width 0.25) (layer "F.Cu") (net 2))
-  (segment (start 4.001 -1.946) (end 3.805 -1.75) (width 0.25) (layer "F.Cu") (net 2))
-  (segment (start -3.501 -1.946) (end -3.42648 -1.87148) (width 0.25) (layer "F.Cu") (net 2))
-  (segment (start 1.313803 -1.87148) (end 1 -2.185283) (width 0.25) (layer "F.Cu") (net 2))
-  (segment (start 0.92548 -1.87148) (end -0.37148 -1.87148) (width 0.25) (layer "F.Cu") (net 2))
-  (segment (start -3.501 -3.396) (end -3.501 -1.946) (width 0.25) (layer "F.Cu") (net 2))
-  (segment (start -2.62852 -1.87148) (end -0.813803 -1.87148) (width 0.25) (layer "F.Cu") (net 2))
-  (segment (start -2.62852 -1.12852) (end -2.5 -1) (width 0.25) (layer "F.Cu") (net 2))
-  (segment (start -0.37148 -1.87148) (end -0.5 -2) (width 0.25) (layer "F.Cu") (net 2))
-  (segment (start 1 -2.185283) (end 1 -3.396) (width 0.25) (layer "F.Cu") (net 2))
-  (segment (start 4.001 -3.396) (end 4.001 -1.946) (width 0.25) (layer "F.Cu") (net 2))
-  (segment (start 2.5 -3.396) (end 2.5 -1.946) (width 0.25) (layer "F.Cu") (net 2))
-  (via (at -2.5 -1) (size 0.8) (drill 0.4) (layers "F.Cu" "B.Cu") (net 2))
-  (segment (start 3.501 -16.499) (end 3.501 -3.396) (width 0.25) (layer "F.Cu") (net 3))
+  (segment (start 5.474511 -4.369511) (end 5.474511 -12.750875) (width 0.25) (layer "F.Cu") (net 1))
+  (segment (start 4.501 -3.396) (end 5.474511 -4.369511) (width 0.25) (layer "F.Cu") (net 1))
+  (segment (start 1 -3.396) (end 1 -7.524598) (width 0.25) (layer "F.Cu") (net 2))
+  (segment (start -3.501 -3.396) (end -3.501 -5.249) (width 0.25) (layer "F.Cu") (net 2))
+  (segment (start 2.5 -6.2755) (end 2.7245 -6.5) (width 0.25) (layer "F.Cu") (net 2))
+  (segment (start -0.5 -5.131316) (end -1.184342 -5.815658) (width 0.25) (layer "F.Cu") (net 2))
+  (segment (start 4.001 -3.396) (end 4.001 -4.846) (width 0.25) (layer "F.Cu") (net 2))
+  (segment (start 1 -7.524598) (end 0.137299 -8.387299) (width 0.25) (layer "F.Cu") (net 2))
+  (segment (start 4.001 -4.846) (end 4.75 -5.595) (width 0.25) (layer "F.Cu") (net 2))
+  (segment (start -0.5 -3.396) (end -0.5 -5.131316) (width 0.25) (layer "F.Cu") (net 2))
+  (segment (start 4.75 -5.595) (end 4.75 -6.5) (width 0.25) (layer "F.Cu") (net 2))
+  (segment (start 2.5 -3.396) (end 2.5 -6.2755) (width 0.25) (layer "F.Cu") (net 2))
+  (via (at -3.501 -5.249) (size 0.8) (drill 0.4) (layers "F.Cu" "B.Cu") (net 2))
+  (via (at -1.184342 -5.815658) (size 0.8) (drill 0.4) (layers "F.Cu" "B.Cu") (net 2))
+  (via (at 2.7245 -6.5) (size 0.8) (drill 0.4) (layers "F.Cu" "B.Cu") (net 2))
+  (via (at 0.137299 -8.387299) (size 0.8) (drill 0.4) (layers "F.Cu" "B.Cu") (net 2))
+  (via (at 4.75 -6.5) (size 0.8) (drill 0.4) (layers "F.Cu" "B.Cu") (net 2))
+  (segment (start 3.5 -7.585238) (end 3.898531 -7.186707) (width 0.25) (layer "F.Cu") (net 3))
+  (segment (start 3.501 -5.001) (end 3.501 -3.396) (width 0.25) (layer "F.Cu") (net 3))
   (segment (start 3.5 -16.5) (end 3.501 -16.499) (width 0.25) (layer "F.Cu") (net 3))
+  (segment (start 3.5 -16.5) (end 3.5 -7.585238) (width 0.25) (layer "F.Cu") (net 3))
+  (segment (start 3.898531 -5.398531) (end 3.501 -5.001) (width 0.25) (layer "F.Cu") (net 3))
+  (segment (start 3.898531 -7.186707) (end 3.898531 -5.398531) (width 0.25) (layer "F.Cu") (net 3))
+  (segment (start 3.449011 -6.199897) (end 3.449011 -7.000509) (width 0.25) (layer "F.Cu") (net 4))
+  (segment (start 3.001 -3.396) (end 3.001 -5.751886) (width 0.25) (layer "F.Cu") (net 4))
   (segment (start 6 -16) (end 5.5 -16.5) (width 0.25) (layer "F.Cu") (net 4))
-  (segment (start 3.001 -3.396) (end 3.001 -5.7235) (width 0.25) (layer "F.Cu") (net 4))
-  (segment (start 3.001 -5.7235) (end 2.7245 -6) (width 0.25) (layer "F.Cu") (net 4))
+  (segment (start 2.69952 -7.75) (end 2.69952 -9.94952) (width 0.25) (layer "F.Cu") (net 4))
+  (segment (start 2.69952 -9.94952) (end 2.7245 -9.9745) (width 0.25) (layer "F.Cu") (net 4))
+  (segment (start 3.001 -5.751886) (end 3.449011 -6.199897) (width 0.25) (layer "F.Cu") (net 4))
+  (segment (start 3.449011 -7.000509) (end 2.69952 -7.75) (width 0.25) (layer "F.Cu") (net 4))
   (segment (start 6 -13.25) (end 6 -16) (width 0.25) (layer "F.Cu") (net 4))
-  (via (at 2.7245 -6) (size 0.8) (drill 0.4) (layers "F.Cu" "B.Cu") (net 4))
+  (via (at 2.7245 -9.9745) (size 0.8) (drill 0.4) (layers "F.Cu" "B.Cu") (net 4))
   (via (at 6 -13.25) (size 0.8) (drill 0.4) (layers "F.Cu" "B.Cu") (net 4))
-  (segment (start 2.7245 -6) (end 2.7245 -9.9745) (width 0.25) (layer "B.Cu") (net 4))
   (segment (start 2.7245 -9.9745) (end 6 -13.25) (width 0.25) (layer "B.Cu") (net 4))
   (segment (start 2.5 -16.5) (end 2 -16) (width 0.25) (layer "F.Cu") (net 5))
   (segment (start 2 -16) (end 2 -3.396) (width 0.25) (layer "F.Cu") (net 5))
-  (segment (start -3.5 -11.635718) (end 1.5 -6.635718) (width 0.25) (layer "F.Cu") (net 6))
-  (segment (start -3.5 -16.5) (end -3.5 -11.635718) (width 0.25) (layer "F.Cu") (net 6))
-  (segment (start 1.5 -6.635718) (end 1.5 -3.396) (width 0.25) (layer "F.Cu") (net 6))
+  (segment (start 1.5 -8.049212) (end -2.086506 -11.635718) (width 0.25) (layer "F.Cu") (net 6))
+  (segment (start -3.5 -11.635718) (end -3.5 -16.5) (width 0.25) (layer "F.Cu") (net 6))
+  (segment (start 1.5 -3.396) (end 1.5 -8.049212) (width 0.25) (layer "F.Cu") (net 6))
+  (segment (start -2.086506 -11.635718) (end -3.5 -11.635718) (width 0.25) (layer "F.Cu") (net 6))
   (segment (start 0.5 -7) (end 0.5 -3.396) (width 0.25) (layer "F.Cu") (net 7))
   (segment (start -4.5 -12) (end 0.5 -7) (width 0.25) (layer "F.Cu") (net 7))
   (segment (start -4.5 -16.5) (end -4.5 -12) (width 0.25) (layer "F.Cu") (net 7))
-  (segment (start 0 -3.396) (end 0 -4.75) (width 0.25) (layer "F.Cu") (net 8))
-  (segment (start 0 -4.75) (end -1.75 -6.5) (width 0.25) (layer "F.Cu") (net 8))
   (segment (start -1.75 -14.5) (end -1.75 -16) (width 0.25) (layer "F.Cu") (net 8))
   (segment (start -2.25 -16.5) (end -2.5 -16.5) (width 0.25) (layer "F.Cu") (net 8))
   (segment (start -1.75 -16) (end -2.25 -16.5) (width 0.25) (layer "F.Cu") (net 8))
-  (via (at -1.75 -6.5) (size 0.8) (drill 0.4) (layers "F.Cu" "B.Cu") (net 8))
+  (segment (start 0 -6.475402) (end -1.887299 -8.362701) (width 0.25) (layer "F.Cu") (net 8))
+  (segment (start 0 -3.396) (end 0 -6.475402) (width 0.25) (layer "F.Cu") (net 8))
+  (via (at -1.887299 -8.362701) (size 0.8) (drill 0.4) (layers "F.Cu" "B.Cu") (net 8))
   (via (at -1.75 -14.5) (size 0.8) (drill 0.4) (layers "F.Cu" "B.Cu") (net 8))
-  (segment (start -1.75 -6.5) (end -1.75 -14.5) (width 0.25) (layer "B.Cu") (net 8))
+  (segment (start -1.887299 -8.362701) (end -1.887299 -14.362701) (width 0.25) (layer "B.Cu") (net 8))
+  (segment (start -1.887299 -14.362701) (end -1.75 -14.5) (width 0.25) (layer "B.Cu") (net 8))
   (segment (start -5.5 -16.5) (end -5.5 -9.106717) (width 0.25) (layer "F.Cu") (net 9))
   (segment (start -1 -4.606717) (end -1 -3.396) (width 0.25) (layer "F.Cu") (net 9))
