File: HDMI_to_Stemma/21Pin_Fanout_Diodes/21Pin_Fanout.kicad_pcb (KiCad board)
At the start: 2 copper layers, 33.8 x 29.5 mm, 5 parts, among them J1 HDMI_A, J6 Conn_01x04, J7 Conn_01x04, J8 Conn_01x04, J9 Conn_01x04

Commit message: Updated traces
Routing:
- net GND: track 19.5 -> 33.7 mm, vias 1 -> 5
- net Net-(J1-Pad10): track 19.6 -> 21.7 mm
- net Net-(J1-Pad12): track 20.1 -> 21.1 mm
