File: HDMI_to_Stemma/21Pin_Fanout_Diodes_&_Heater/21Pin_Fanout.kicad_pcb (KiCad board)
At the start: 2 copper layers, 33.8 x 31 mm, 5 parts, among them J1 HDMI_A, J2 Conn_01x02, J3 Conn_01x02, J6 Conn_01x04, J7 Conn_01x04

Commit message: Updated traces
Routing:
- net GND: track 19.9 -> 30.5 mm, vias 1 -> 5
- net Net-(J1-Pad10): track 20.4 -> 21.0 mm
Changed lines of the file:
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@@
     (effects (font (size 0.5 0.5) (thickness 0.125)) (justify mirror))
   )
-  (segment (start 4.501 -11.001) (end 11.05048 -17.55048) (width 0.25) (layer "F.Cu") (net 1))
-  (segment (start 4.501 -3.396) (end 4.501 -11.001) (width 0.25) (layer "F.Cu") (net 1))
+  (segment (start 5.5 -12) (end 11.05048 -17.55048) (width 0.25) (layer "F.Cu") (net 1))
   (segment (start 13.32596 -17.55048) (end 14.15 -18.37452) (width 0.25) (layer "F.Cu") (net 1))
+  (segment (start 4.501 -3.396) (end 4.501 -6.251) (width 0.25) (layer "F.Cu") (net 1))
   (segment (start 11.05048 -17.55048) (end 13.32596 -17.55048) (width 0.25) (layer "F.Cu") (net 1))
+  (segment (start 5 -6.75) (end 5 -11.5) (width 0.25) (layer "F.Cu") (net 1))
+  (segment (start 5 -11.5) (end 5.5 -12) (width 0.25) (layer "F.Cu") (net 1))
   (segment (start 14.15 -18.37452) (end 14.15 -19.25) (width 0.25) (layer "F.Cu") (net 1))
-  (segment (start 1 -1.946) (end 0.92548 -1.87148) (width 0.25) (layer "F.Cu") (net 2))
-  (segment (start 4.001 -3.396) (end 4.001 -1.946) (width 0.25) (layer "F.Cu") (net 2))
-  (segment (start -2.12852 -1.87148) (end -2.12852 -0.87148) (width 0.25) (layer "F.Cu") (net 2))
-  (segment (start 2.5 -2.186283) (end 2.5 -3.396) (width 0.25) (layer "F.Cu") (net 2))
-  (segment (start -0.37148 -1.87148) (end -0.5 -2) (width 0.25) (layer "F.Cu") (net 2))
-  (segment (start -0.5 -1.946) (end -0.57452 -1.87148) (width 0.25) (layer "F.Cu") (net 2))
-  (segment (start -0.5 -2) (end -0.5 -3.396) (width 0.25) (layer "F.Cu") (net 2))
-  (segment (start 1 -3.396) (end 1 -1.946) (width 0.25) (layer "F.Cu") (net 2))
-  (segment (start -0.57452 -1.87148) (end -2.12852 -1.87148) (width 0.25) (layer "F.Cu") (net 2))
-  (segment (start 2.5 -1.946) (end 2.42548 -1.87148) (width 0.25) (layer "F.Cu") (net 2))
-  (segment (start 1.313803 -1.87148) (end 1 -2.185283) (width 0.25) (layer "F.Cu") (net 2))
-  (segment (start 2.814803 -1.87148) (end 2.5 -2.186283) (width 0.25) (layer "F.Cu") (net 2))
-  (segment (start -2.12852 -1.87148) (end -3.187197 -1.87148) (width 0.25) (layer "F.Cu") (net 2))
-  (segment (start 4.001 -1.946) (end 3.92648 -1.87148) (width 0.25) (layer "F.Cu") (net 2))
-  (segment (start 2.42548 -1.87148) (end 1.313803 -1.87148) (width 0.25) (layer "F.Cu") (net 2))
-  (segment (start -0.5 -3.396) (end -0.5 -1.946) (width 0.25) (layer "F.Cu") (net 2))
-  (segment (start 0.92548 -1.87148) (end -0.37148 -1.87148) (width 0.25) (layer "F.Cu") (net 2))
-  (segment (start 1 -2.185283) (end 1 -3.396) (width 0.25) (layer "F.Cu") (net 2))
-  (segment (start -3.501 -2.185283) (end -3.501 -3.396) (width 0.25) (layer "F.Cu") (net 2))
-  (segment (start 2.5 -3.396) (end 2.5 -1.946) (width 0.25) (layer "F.Cu") (net 2))
-  (segment (start -3.187197 -1.87148) (end -3.501 -2.185283) (width 0.25) (layer "F.Cu") (net 2))
-  (segment (start 3.92648 -1.87148) (end 2.814803 -1.87148) (width 0.25) (layer "F.Cu") (net 2))
-  (via (at -2.12852 -0.87148) (size 0.8) (drill 0.4) (layers "F.Cu" "B.Cu") (net 2))
+  (segment (start 4.501 -6.251) (end 5 -6.75) (width 0.25) (layer "F.Cu") (net 1))
+  (segment (start -0.5 -7.951402) (end -2.899299 -10.350701) (width 0.25) (layer "F.Cu") (net 2))
+  (segment (start 4.001 -3.396) (end 4.001 -7.0255) (width 0.25) (layer "F.Cu") (net 2))
+  (segment (start -3.501 -5.499) (end -3.5 -5.5) (width 0.25) (layer "F.Cu") (net 2))
+  (segment (start 2.5 -3.396) (end 2.5 -11.7755) (width 0.25) (layer "F.Cu") (net 2))
+  (segment (start 1 -3.396) (end 1 -9.136332) (width 0.25) (layer "F.Cu") (net 2))
+  (segment (start -0.5 -3.396) (end -0.5 -7.951402) (width 0.25) (layer "F.Cu") (net 2))
+  (segment (start 4.001 -7.0255) (end 4.2255 -7.25) (width 0.25) (layer "F.Cu") (net 2))
+  (segment (start 2.5 -11.7755) (end 2.7245 -12) (width 0.25) (layer "F.Cu") (net 2))
+  (segment (start -3.501 -3.396) (end -3.501 -5.499) (width 0.25) (layer "F.Cu") (net 2))
+  (segment (start 1 -9.136332) (end -0.431834 -10.568166) (width 0.25) (layer "F.Cu") (net 2))
+  (via (at 2.7245 -12) (size 0.8) (drill 0.4) (layers "F.Cu" "B.Cu") (net 2))
+  (via (at -3.5 -5.5) (size 0.8) (drill 0.4) (layers "F.Cu" "B.Cu") (net 2))
+  (via (at -0.431834 -10.568166) (size 0.8) (drill 0.4) (layers "F.Cu" "B.Cu") (net 2))
+  (via (at 4.2255 -7.25) (size 0.8) (drill 0.4) (layers "F.Cu" "B.Cu") (net 2))
+  (via (at -2.899299 -10.350701) (size 0.8) (drill 0.4) (layers "F.Cu" "B.Cu") (net 2))
   (segment (start 13 -18) (end 13 -19.1) (width 0.25) (layer "F.Cu") (net 3))
+  (segment (start 3.898531 -16.166741) (end 4.240895 -16.509105) (width 0.25) (layer "F.Cu") (net 3))
   (segment (start 13 -19.1) (end 13.15 -19.25) (width 0.25) (layer "F.Cu") (net 3))
-  (segment (start 3.501 -3.396) (end 3.501 -15.76921) (width 0.25) (layer "F.Cu") (net 3))
+  (segment (start 3.898531 -11.5137) (end 3.898531 -16.166741) (width 0.25) (layer "F.Cu") (net 3))
   (segment (start 5.73179 -18) (end 13 -18) (width 0.25) (layer "F.Cu") (net 3))
-  (segment (start 3.501 -15.76921) (end 5.73179 -18) (width 0.25) (layer "F.Cu") (net 3))
+  (segment (start 3.501 -11.116168) (end 3.898531 -11.5137) (width 0.25) (layer "F.Cu") (net 3))
+  (segment (start 4.240895 -16.509105) (end 5.73179 -18) (width 0.25) (layer "F.Cu") (net 3))
+  (segment (start 3.501 -3.396) (end 3.501 -11.116168) (width 0.25) (layer "F.Cu") (net 3))
+  (segment (start 3.449011 -11.699897) (end 3.449011 -12.300989) (width 0.25) (layer "F.Cu") (net 4))
+  (segment (start 3 -12.75) (end 3 -15.903928) (width 0.25) (layer "F.Cu") (net 4))
   (segment (start 5.9 -18.803928) (end 5.9 -19.25) (width 0.25) (layer "F.Cu") (net 4))
-  (segment (start 3.001 -3.396) (end 3.001 -15.904928) (width 0.25) (layer "F.Cu") (net 4))
-  (segment (start 3.001 -15.904928) (end 5.9 -18.803928) (width 0.25) (layer "F.Cu") (net 4))
-  (segment (start 4.9 -18.803928) (end 4.9 -19.25) (width 0.25) (layer "F.Cu") (net 5))
+  (segment (start 3.001 -11.251886) (end 3.449011 -11.699897) (width 0.25) (layer "F.Cu") (net 4))
+  (segment (start 3.001 -3.396) (end 3.001 -11.251886) (width 0.25) (layer "F.Cu") (net 4))
+  (segment (start 3.449011 -12.300989) (end 3 -12.75) (width 0.25) (layer "F.Cu") (net 4))
+  (segment (start 3 -15.903928) (end 5.9 -18.803928) (width 0.25) (layer "F.Cu") (net 4))
   (segment (start 2 -15.903928) (end 4.9 -18.803928) (width 0.25) (layer "F.Cu") (net 5))
   (segment (start 2 -3.396) (end 2 -15.903928) (width 0.25) (layer "F.Cu") (net 5))
-  (segment (start 1.5 -3.396) (end 1.5 -8.385717) (width 0.25) (layer "F.Cu") (net 6))
-  (segment (start -2.25 -12.135717) (end -2.25 -19.25) (width 0.25) (layer "F.Cu") (net 6))
-  (segment (start 1.5 -8.385717) (end -2.25 -12.135717) (width 0.25) (layer "F.Cu") (net 6))
-  (segment (start -4.25 -13.185718) (end -4.25 -19.25) (width 0.25) (layer "F.Cu") (net 7))
-  (segment (start 0.185718 -8.75) (end -4.25 -13.185718) (width 0.25) (layer "F.Cu") (net 7))
-  (segment (start 0.5 -3.396) (end 0.5 -8.75) (width 0.25) (layer "F.Cu") (net 7))
-  (segment (start 0.5 -8.75) (end 0.185718 -8.75) (width 0.25) (layer "F.Cu") (net 7))
-  (segment (start 0 -8.3) (end -10.95 -19.25) (width 0.25) (layer "F.Cu") (net 8))
-  (segment (start 0 -3.396) (end 0 -8.3) (width 0.25) (layer "F.Cu") (net 8))
-  (segment (start -1 -7.426804) (end -1 -3.396) (width 0.25) (layer "F.Cu") (net 9))
-  (segment (start -12.823196 -19.25) (end -1 -7.426804) (width 0.25) (layer "F.Cu") (net 9))
-  (segment (start -12.95 -19.25) (end -12.823196 -19.25) (width 0.25) (layer "F.Cu") (net 9))
+  (segment (start 4.9 -18.803928) (end 4.9 -19.25) (width 0.25) (layer "F.Cu") (net 5))
+  (segment (start 1.5 -3.396) (end 1.5 -9.75) (width 0.25) (layer "F.Cu") (net 6))
+  (segment (start -2.5 -13.75) (end -2.5 -19) (width 0.25) (layer "F.Cu") (net 6))
+  (segment (start -2.5 -19) (end -2.25 -19.25) (width 0.25) (layer "F.Cu") (net 6))
+  (segment (start 1.5 -9.75) (end -2.5 -13.75) (width 0.25) (layer "F.Cu") (net 6))
+  (segment (start 0.5 -8.611733) (end -4.25 -13.361733) (width 0.25) (layer "F.Cu") (net 7))
+  (segment (start -4.25 -13.361733) (end -4.25 -14) (width 0.25) (layer "F.Cu") (net 7))
+  (segment (start -4.25 -14) (end -4.25 -19.25) (width 0.25) (layer "F.Cu") (net 7))
+  (segment (start 0.5 -3.396) (end 0.5 -8.611733) (width 0.25) (layer "F.Cu") (net 7))
+  (segment (start -10.95 -18.350424) (end -10.95 -19.25) (width 0.25) (layer "F.Cu") (net 8))
+  (segment (start 0 -8.476016) (end -2.599196 -11.075212) (width 0.25) (layer "F.Cu") (net 8))
+  (segment (start -2.599196 -11.075212) (end -3.674788 -11.075212) (width 0.25) (layer "F.Cu") (net 8))
+  (segment (start -3.674788 -11.075212) (end -10.95 -18.350424) (width 0.25) (layer "F.Cu") (net 8))
+  (segment (start 0 -3.396) (end 0 -8.476016) (width 0.25) (layer "F.Cu") (net 8))
+  (segment (start -12.823196 -19.25) (end -12.95 -19.25) (width 0.25) (layer "F.Cu") (net 9))
+  (segment (start -1 -3.396) (end -1 -7.426804) (width 0.25) (layer "F.Cu") (net 9))
+  (segment (start -1 -7.426804) (end -12.823196 -19.25) (width 0.25) (layer "F.Cu") (net 9))
   (zone (net 2) (net_name "GND") (layer "F.Cu") (hatch edge 0.508)
     (connect_pads (clearance 0.508))
