File: HDMI_to_Stemma/21Pin_Fanout_Heater_&_Extra/21Pin_Fanout.kicad_pcb (KiCad board)
At the start: 2 copper layers, 33.2 x 38.2 mm, 5 parts, among them J1 HDMI_A, J2 Conn_01x02, J3 Conn_01x02, J4 Conn_01x02, J5 Conn_01x02

Commit message: Update
Other:
- board text added: "HDMI_JST_21Pin_Heaters & Extra Ryan Morgenstern 6/62022"
- board text removed: "HDMI_JST_21Pin_Diodes & Heaters Ryan Morgenstern 6/62022"
Changed lines of the file:
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@@
   (gr_line (start -8.5 -4.75) (end -8.5 -14.75) (layer "Edge.Cuts") (width 0.1))
   (gr_line (start 8.5 -4.75) (end 8.5 6.75) (layer "Edge.Cuts") (width 0.1))
-  (gr_text "HDMI_JST_21Pin_Diodes & Heaters\nRyan Morgenstern\n6/62022" (at 0.25 1) (layer "B.SilkS")
+  (gr_text "HDMI_JST_21Pin_Heaters & Extra\nRyan Morgenstern\n6/62022" (at 0.25 1) (layer "B.SilkS")
     (effects (font (size 0.5 0.5) (thickness 0.125)) (justify mirror))
   )

Commit message: Updated traces
Routing:
- net GND: track 19.8 -> 37.5 mm, vias 1 -> 5
- net Net-(J1-Pad4): track 24.5 -> 25.2 mm
- net Net-(J1-Pad3): track 29.0 -> 29.6 mm
Changed lines of the file:
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@@
     (effects (font (size 0.5 0.5) (thickness 0.125)) (justify mirror))
   )
-  (segment (start 14.75 -26.5) (end 11.932141 -23.682141) (width 0.25) (layer "F.Cu") (net 1))
-  (segment (start 4.501 -21.115282) (end 4.501 -3.396) (width 0.25) (layer "F.Cu") (net 1))
-  (segment (start 7.067859 -23.682141) (end 4.501 -21.115282) (width 0.25) (layer "F.Cu") (net 1))
-  (segment (start 11.932141 -23.682141) (end 7.067859 -23.682141) (width 0.25) (layer "F.Cu") (net 1))
-  (segment (start -2.12148 -1.87148) (end -2.12148 -1.12148) (width 0.25) (layer "F.Cu") (net 2))
-  (segment (start -0.813803 -1.87148) (end -0.5 -2.185283) (width 0.25) (layer "F.Cu") (net 2))
-  (segment (start 2.5 -1.946) (end 2.696 -1.75) (width 0.25) (layer "F.Cu") (net 2))
-  (segment (start 1 -1.946) (end 1.07452 -1.87148) (width 0.25) (layer "F.Cu") (net 2))
-  (segment (start 1 -3.396) (end 1 -1.946) (width 0.25) (layer "F.Cu") (net 2))
-  (segment (start -2.12148 -1.87148) (end -0.813803 -1.87148) (width 0.25) (layer "F.Cu") (net 2))
-  (segment (start -3.501 -3.396) (end -3.501 -1.946) (width 0.25) (layer "F.Cu") (net 2))
-  (segment (start -0.5 -1.946) (end -0.42548 -1.87148) (width 0.25) (layer "F.Cu") (net 2))
+  (segment (start 5.009441 -21.623723) (end 7.067859 -23.682141) (width 0.25) (layer "F.Cu") (net 1))
+  (segment (start 5.009441 -3.904441) (end 5.009441 -21.623723) (width 0.25) (layer "F.Cu") (net 1))
+  (segment (start 4.501 -3.396) (end 5.009441 -3.904441) (width 0.25) (layer "F.Cu") (net 1))
+  (segment (start 7.067859 -23.682141) (end 11.932141 -23.682141) (width 0.25) (layer "F.Cu") (net 1))
+  (segment (start 11.932141 -23.682141) (end 14.75 -26.5) (width 0.25) (layer "F.Cu") (net 1))
+  (segment (start 1 -11.0255) (end 1.2245 -11.25) (width 0.25) (layer "F.Cu") (net 2))
+  (segment (start -3.501 -5.999) (end -3.5 -6) (width 0.25) (layer "F.Cu") (net 2))
+  (segment (start 1 -3.396) (end 1 -11.0255) (width 0.25) (layer "F.Cu") (net 2))
+  (segment (start 4.001 -8.65664) (end 4.28493 -8.94057) (width 0.25) (layer "F.Cu") (net 2))
+  (segment (start 2.5 -9.84057) (end 2.829715 -10.170285) (width 0.25) (layer "F.Cu") (net 2))
   (segment (start -0.5 -2.185283) (end -0.5 -3.396) (width 0.25) (layer "F.Cu") (net 2))
-  (segment (start 2.5 -3.396) (end 2.5 -1.946) (width 0.25) (layer "F.Cu") (net 2))
-  (segment (start -3.42648 -1.87148) (end -2.12148 -1.87148) (width 0.25) (layer "F.Cu") (net 2))
+  (segment (start -0.5 -12.5255) (end -0.2755 -12.75) (width 0.25) (layer "F.Cu") (net 2))
+  (segment (start 4.001 -3.396) (end 4.001 -8.65664) (width 0.25) (layer "F.Cu") (net 2))
   (segment (start 4.001 -2.185283) (end 4.001 -3.396) (width 0.25) (layer "F.Cu") (net 2))
-  (segment (start 2.696 -1.75) (end 3.565717 -1.75) (width 0.25) (layer "F.Cu") (net 2))
   (segment (start 1 -2.134803) (end 1 -3.396) (width 0.25) (layer "F.Cu") (net 2))
-  (segment (start 0.736677 -1.87148) (end 1 -2.134803) (width 0.25) (layer "F.Cu") (net 2))
-  (segment (start -2.12148 -1.12148) (end -2 -1) (width 0.25) (layer "F.Cu") (net 2))
-  (segment (start -0.5 -3.396) (end -0.5 -1.946) (width 0.25) (layer "F.Cu") (net 2))
-  (segment (start -3.501 -1.946) (end -3.42648 -1.87148) (width 0.25) (layer "F.Cu") (net 2))
-  (segment (start -0.42548 -1.87148) (end 0.736677 -1.87148) (width 0.25) (layer "F.Cu") (net 2))
-  (segment (start 2.186197 -1.87148) (end 2.5 -2.185283) (width 0.25) (layer "F.Cu") (net 2))
+  (segment (start -0.5 -3.396) (end -0.5 -12.5255) (width 0.25) (layer "F.Cu") (net 2))
+  (segment (start -3.501 -3.396) (end -3.501 -5.999) (width 0.25) (layer "F.Cu") (net 2))
   (segment (start 2.5 -2.185283) (end 2.5 -3.396) (width 0.25) (layer "F.Cu") (net 2))
-  (segment (start 1.07452 -1.87148) (end 2.186197 -1.87148) (width 0.25) (layer "F.Cu") (net 2))
-  (segment (start 3.565717 -1.75) (end 4.001 -2.185283) (width 0.25) (layer "F.Cu") (net 2))
-  (via (at -2 -1) (size 0.8) (drill 0.4) (layers "F.Cu" "B.Cu") (net 2))
-  (segment (start 3.501 -3.396) (end 3.501 -20.751) (width 0.25) (layer "F.Cu") (net 3))
-  (segment (start 3.501 -20.751) (end 9.25 -26.5) (width 0.25) (layer "F.Cu") (net 3))
+  (segment (start 2.5 -3.396) (end 2.5 -9.84057) (width 0.25) (layer "F.Cu") (net 2))
+  (via (at 2.829715 -10.170285) (size 0.8) (drill 0.4) (layers "F.Cu" "B.Cu") (net 2))
+  (via (at -3.5 -6) (size 0.8) (drill 0.4) (layers "F.Cu" "B.Cu") (net 2))
+  (via (at 4.28493 -8.94057) (size 0.8) (drill 0.4) (layers "F.Cu" "B.Cu") (net 2))
+  (via (at 1.2245 -11.25) (size 0.8) (drill 0.4) (layers "F.Cu" "B.Cu") (net 2))
+  (via (at -0.2755 -12.75) (size 0.8) (drill 0.4) (layers "F.Cu" "B.Cu") (net 2))
+  (segment (start 4.19952 -9.879758) (end 4.19952 -13.05048) (width 0.25) (layer "F.Cu") (net 3))
+  (segment (start 3.5 -13.75) (end 3.5 -20.75) (width 0.25) (layer "F.Cu") (net 3))
+  (segment (start 3.501 -9.181238) (end 4.19952 -9.879758) (width 0.25) (layer "F.Cu") (net 3))
+  (segment (start 3.5 -20.75) (end 9.25 -26.5) (width 0.25) (layer "F.Cu") (net 3))
   (segment (start 9.25 -26.5) (end 12.75 -26.5) (width 0.25) (layer "F.Cu") (net 3))
-  (segment (start 3.001 -23.051) (end 3.001 -3.396) (width 0.25) (layer "F.Cu") (net 4))
-  (segment (start 6.45 -26.5) (end 3.001 -23.051) (width 0.25) (layer "F.Cu") (net 4))
-  (segment (start 2 -3.396) (end 2 -24.05) (width 0.25) (layer "F.Cu") (net 5))
-  (segment (start 2 -24.05) (end 4.45 -26.5) (width 0.25) (layer "F.Cu") (net 5))
+  (segment (start 4.19952 -13.05048) (end 3.5 -13.75) (width 0.25) (layer "F.Cu") (net 3))
+  (segment (start 3.501 -3.396) (end 3.501 -9.181238) (width 0.25) (layer "F.Cu") (net 3))
+  (segment (start 3 -23.05) (end 6.45 -26.5) (width 0.25) (layer "F.Cu") (net 4))
+  (segment (start 3 -11.5) (end 3 -23.05) (width 0.25) (layer "F.Cu") (net 4))
+  (segment (start 3.75 -10.065956) (end 3.75 -10.75) (width 0.25) (layer "F.Cu") (net 4))
+  (segment (start 3.001 -3.396) (end 3.001 -9.316956) (width 0.25) (layer "F.Cu") (net 4))
+  (segment (start 3.75 -10.75) (end 3 -11.5) (width 0.25) (layer "F.Cu") (net 4))
+  (segment (start 3.001 -9.316956) (end 3.75 -10.065956) (width 0.25) (layer "F.Cu") (net 4))
+  (segment (start 2 -10.365168) (end 2.5 -10.865168) (width 0.25) (layer "F.Cu") (net 5))
+  (segment (start 1.94952 -12.30048) (end 1.94952 -23.99952) (width 0.25) (layer "F.Cu") (net 5))
+  (segment (start 1.94952 -23.99952) (end 4.45 -26.5) (width 0.25) (layer "F.Cu") (net 5))
+  (segment (start 2.5 -11.75) (end 1.94952 -12.30048) (width 0.25) (layer "F.Cu") (net 5))
+  (segment (start 2.5 -10.865168) (end 2.5 -11.75) (width 0.25) (layer "F.Cu") (net 5))
+  (segment (start 2 -3.396) (end 2 -10.365168) (width 0.25) (layer "F.Cu") (net 5))
+  (segment (start 1.5 -10.500886) (end 1.5 -3.396) (width 0.25) (layer "F.Cu") (net 6))
   (segment (start -2 -26.5) (end 1.5 -23) (width 0.25) (layer "F.Cu") (net 6))
-  (segment (start 1.5 -23) (end 1.5 -3.396) (width 0.25) (layer "F.Cu") (net 6))
-  (segment (start -4 -26.5) (end 0.5 -22) (width 0.25) (layer "F.Cu") (net 7))
-  (segment (start 0.5 -22) (end 0.5 -3.396) (width 0.25) (layer "F.Cu") (net 7))
-  (segment (start 0 -16.05) (end -10.45 -26.5) (width 0.25) (layer "F.Cu") (net 8))
-  (segment (start 0 -3.396) (end 0 -16.05) (width 0.25) (layer "F.Cu") (net 8))
-  (segment (start -1 -15.05) (end -1 -3.396) (width 0.25) (layer "F.Cu") (net 9))
+  (segment (start 1.949011 -10.949897) (end 1.5 -10.500886) (width 0.25) (layer "F.Cu") (net 6))
+  (segment (start 1.5 -12.098051) (end 1.949011 -11.64904) (width 0.25) (layer "F.Cu") (net 6))
+  (segment (start 1.949011 -11.64904) (end 1.949011 -10.949897) (width 0.25) (layer "F.Cu") (net 6))
+  (segment (start 1.5 -23) (end 1.5 -12.098051) (width 0.25) (layer "F.Cu") (net 6))
+  (segment (start 0.5 -3.396) (end 0.5 -11.664762) (width 0.25) (layer "F.Cu") (net 7))
+  (segment (start 0.898531 -12.063293) (end 0.898531 -21.601469) (width 0.25) (layer "F.Cu") (net 7))
+  (segment (start 0.898531 -21.601469) (end -4 -26.5) (width 0.25) (layer "F.Cu") (net 7))
+  (segment (start 0.5 -11.664762) (end 0.898531 -12.063293) (width 0.25) (layer "F.Cu") (net 7))
+  (segment (start 0 -11.80048) (end 0 -3.396) (width 0.25) (layer "F.Cu") (net 8))
+  (segment (start 0.449011 -12.249491) (end 0 -11.80048) (width 0.25) (layer "F.Cu") (net 8))
+  (segment (start 0.449011 -15.600989) (end 0.449011 -12.249491) (width 0.25) (layer "F.Cu") (net 8))
+  (segment (start -10.45 -26.5) (end 0.449011 -15.600989) (width 0.25) (layer "F.Cu") (net 8))
+  (segment (start -1 -3.396) (end -1 -15.05) (width 0.25) (layer "F.Cu") (net 9))
   (segment (start -12.45 -26.5) (end -1 -15.05) (width 0.25) (layer "F.Cu") (net 9))
   (zone (net 2) (net_name "GND") (layer "F.Cu") (hatch edge 0.508)
